File: kicad/soc.kicad_pcb (KiCad board)
At the start: 2 copper layers, 104.1 x 63.5 mm, 18 parts, among them J1 Line Out, J2 PS/2 Keyboard, J3 PS/2 Mouse, J4 Line In, P1 LED MATRIX, P10 CODEC right, P2 ALTERA_DE1_GPIO, P3 Bluetooth, P4 CONN_01X08, P9 CODEC left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

Commit message: more board tweaks
Parts:
- moved P4 20.9 mm to (77.5, 97.8), turned to 90 degrees
- moved U2 12.8 mm to (61.0, 100.3)
- moved P1 2.54 mm to (57.1, 68.6)
Routing:
- net +5V: track 0.00 -> 120.4 mm
- net /Kbd_data: track 0.00 -> 99.8 mm
- net /Mouse_data: track 0.00 -> 97.7 mm
- net /Kbd_clk: track 0.00 -> 94.4 mm
- net /Mouse_clk: track 0.00 -> 92.6 mm
- net /~CODEC_XDCS: track 0.00 -> 88.0 mm
- net /CODEC_DIRQ: track 0.00 -> 69.0 mm
- net /CODEC_MOSI: track 0.00 -> 68.7 mm
- net /~CODEC_CS: track 0.00 -> 68.7 mm
- net /CODEC_SCLK: track 0.00 -> 66.5 mm
- net /~RST: track 0.00 -> 66.3 mm
- net /CODEC_MISO: track 0.00 -> 64.9 mm
- net /IO_20: track 0.00 -> 61.6 mm
- net /MOSI_33: track 0.00 -> 54.3 mm
- net /MISO_33: track 0.00 -> 50.4 mm
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- added copper zone on B.Cu, net GND
- added copper zone on F.Cu, net GND
- added copper zone on B.Cu, net GNDA
- added copper zone on F.Cu, net GNDA

Commit message: updates to support board
Parts:
- P4: value CONN_01X08 -> CONN_01X09; footprint Pin_Headers:Pin_Header_Straight_2x04 -> Pin_Headers:Pin_Header_Straight_1x09
- moved P4 6.84 mm to (71.1, 95.2)
Connections:
- J2 pad 2: Net-(J2-Pad2) -> (no net)
- J2 pad 6: Net-(J2-Pad6) -> (no net)
- J3 pad 2: Net-(J3-Pad2) -> (no net)
- J3 pad 6: Net-(J3-Pad6) -> (no net)
- P1 pad 12: Net-(P1-Pad12) -> (no net)
- P10 pad 1: Net-(P10-Pad1) -> (no net)
- P10 pad 10: Net-(P10-Pad10) -> (no net)
- P10 pad 11: Net-(P10-Pad11) -> (no net)
- P10 pad 12: Net-(P10-Pad12) -> (no net)
- P10 pad 14: Net-(P10-Pad14) -> (no net)
- P10 pad 2: Net-(P10-Pad2) -> (no net)
- P10 pad 3: Net-(P10-Pad3) -> (no net)
- P10 pad 4: Net-(P10-Pad4) -> (no net)
- P10 pad 5: Net-(P10-Pad5) -> (no net)
- P10 pad 6: Net-(P10-Pad6) -> (no net)
- P10 pad 7: Net-(P10-Pad7) -> (no net)
- P10 pad 8: Net-(P10-Pad8) -> (no net)
- P10 pad 9: Net-(P10-Pad9) -> (no net)
- P3 pad 6: /BLE_DEV -> (no net)
- P4 pad 1: /IO_17 -> /Serial1
- P4 pad 2: /IO_19 -> /IO_17
- P4 pad 3: /IO_20 -> /IO_19
- P4 pad 4: /IO_30 -> /IO_20
- P4 pad 5: /IO_31 -> /IO_30
- P4 pad 6: /IO_32 -> /IO_31
- P4 pad 7: +3V3 -> /IO_32
- P4 pad 8: GND -> +3V3
- P9 pad 2: Net-(P9-Pad2) -> (no net)
- P9 pad 9: Net-(P9-Pad9) -> (no net)
- U2 pad 10: Net-(U2-Pad10) -> (no net)
- U2 pad 11: Net-(U2-Pad11) -> (no net)
- U2 pad 12: Net-(U2-Pad12) -> (no net)
- U2 pad 13: Net-(U2-Pad13) -> (no net)
- U2 pad 14: Net-(U2-Pad14) -> (no net)
- U2 pad 2: Net-(U2-Pad2) -> (no net)
- U2 pad 3: Net-(U2-Pad3) -> (no net)
- U2 pad 5: Net-(U2-Pad5) -> (no net)
- U2 pad 6: Net-(U2-Pad6) -> (no net)
- U2 pad 7: Net-(U2-Pad7) -> (no net)
- U2 pad 8: Net-(U2-Pad8) -> (no net)
- U2 pad 9: Net-(U2-Pad9) -> (no net)
Routing:
- net /IO_20: track 61.6 -> 0.37 mm
- net /IO_17: track 49.8 -> 0.00 mm
- net GND: track 0.00 -> 11.2 mm
- net +3V3: track 43.0 -> 49.8 mm
- net /CODEC_MOSI: track 68.7 -> 74.6 mm
- net /CODEC_SCLK: track 66.5 -> 72.2 mm
- net /CODEC_MISO: track 64.9 -> 70.1 mm
- net /IO_31: track 40.3 -> 43.9 mm
- net /IO_30: track 41.6 -> 44.6 mm
- net /IO_19: track 29.7 -> 28.5 mm
- net /IO_32: track 48.6 -> 49.5 mm
