File: kicad/soc.sch (KiCad schematic (older format))
At the start: 64 parts, among them J1 Line Out, J2 PS/2 Keyboard, J3 DB9, J4 Line In, J5 Headphone, P1 LED MATRIX, P2 ALTERA_DE1_GPIO, P3 IO, U1 SSM2603, U2 DS3234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

Commit message: incorporate io board serial port as port 2, fix up SPI to be able to support an additional slave select on the io board, working forimware for the 7seg board, and small fixups for the IO board schematic and layout.  this shouldn't be one commit but it kind of just all happened at once.
Parts:
- D3: value TX0 -> RX2
- D4: value RX0 -> TX2
Connections:
- no-connect marks 17 -> 13
Other:
- moved on the sheet: D1, D2, D3, D4, J2, P1, P3, R12, R15, R16, R17, R18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

Commit message: start of IO board adjustments to use USB instead of serial
Parts:
- removed C19, C20, C21, C22, C23: 0.1uF, Capacitors_SMD:C_0805_HandSoldering, symbol C
- removed J3: DB9, mstock-pretty:DB9F, symbol DB9
- removed U4: MAX3232, mstock-pretty:SOIC-16, symbol MAX3232
- BT1: symbol Battery -> Battery-RESCUE-soc
Connections:
- wire segments 165 -> 144
- no-connect marks 13 -> 9
Changed lines of the file:
@@
 EESchema Schematic File Version 2
+LIBS:soc-rescue
 LIBS:power
 LIBS:device
@@
 NoConn ~ 5000 1350
 $Comp
-L Battery BT1
+L Battery-RESCUE-soc BT1
 U 1 1 5699741B
 P 6450 1500
@@
 	5750 4950 5750 5350
 $Comp
-L MAX3232 U4
-U 1 1 585161D1
-P 2000 6150
-F 0 "U4" H 2000 7117 50  0000 C CNN
-F 1 "MAX3232" H 2000 7026 50  0000 C CNN
-F 2 "mstock-pretty:SOIC-16" H 2000 6150 50  0001 C CNN
-F 3 "" H 2000 6150 50  0000 C CNN
-	1    2000 6150
-	1    0    0    -1
-$EndComp
-$Comp
-L C C19
-U 1 1 5851638D
-P 1200 5650
-F 0 "C19" H 1315 5696 50  0000 L CNN
-F 1 "0.1uF" H 1315 5605 50  0000 L CNN
-F 2 "Capacitors_SMD:C_0805_HandSoldering" H 1238 5500 50  0001 C CNN
-F 3 "" H 1200 5650 50  0000 C CNN
-	1    1200 5650
-	1    0    0    -1
-$EndComp
-$Comp
-L C C20
-U 1 1 58516679
-P 1200 6150
-F 0 "C20" H 1315 6196 50  0000 L CNN
-F 1 "0.1uF" H 1315 6105 50  0000 L CNN
-F 2 "Capacitors_SMD:C_0805_HandSoldering" H 1238 6000 50  0001 C CNN
-F 3 "" H 1200 6150 50  0000 C CNN
-	1    1200 6150
-	1    0    0    -1
-$EndComp
-$Comp
-L C C23
-U 1 1 58516739
-P 2850 6350
-F 0 "C23" V 2598 6350 50  0000 C CNN
-F 1 "0.1uF" V 2689 6350 50  0000 C CNN
-F 2 "Capacitors_SMD:C_0805_HandSoldering" H 2888 6200 50  0001 C CNN
-F 3 "" H 2850 6350 50  0000 C CNN
-	1    2850 6350
-	0    1    1    0
-$EndComp
-Wire Wire Line
-	1200 5800 1200 5850
-Wire Wire Line
-	1200 5850 1400 5850
-Wire Wire Line
-	1400 5950 1200 5950
-Wire Wire Line
-	1200 5950 1200 6000
-Wire Wire Line
-	1200 6300 1200 6350
-Wire Wire Line
-	1200 6350 1400 6350
-Wire Wire Line
-	1200 5500 1200 5450
-Wire Wire Line
-	1200 5450 1400 5450
-$Comp
-L GND #PWR029
-U 1 1 58516EE1
-P 3400 6050
-F 0 "#PWR029" H 3400 5800 50  0001 C CNN
-F 1 "GND" H 3400 5900 50  0000 C CNN
-F 2 "" H 3400 6050 60  0000 C CNN
-F 3 "" H 3400 6050 60  0000 C CNN
-	1    3400 6050
-	1    0    0    -1
-$EndComp
-$Comp
-L +3.3V #PWR030
-U 1 1 585175F5
-P 2600 5350
-F 0 "#PWR030" H 2600 5200 50  0001 C CNN
-F 1 "+3.3V" H 2600 5490 50  0000 C CNN
-F 2 "" H 2600 5350 60  0000 C CNN
-F 3 "" H 2600 5350 60  0000 C CNN
-	1    2600 5350
-	1    0    0    -1
-$EndComp
-$Comp
-L C C22
-U 1 1 58517C74
-P 2850 5850
-F 0 "C22" V 2598 5850 50  0000 C CNN
-F 1 "0.1uF" V 2689 5850 50  0000 C CNN
-F 2 "Capacitors_SMD:C_0805_HandSoldering" H 2888 5700 50  0001 C CNN
-F 3 "" H 2850 5850 50  0000 C CNN
-	1    2850 5850
-	0    1    1    0
-$EndComp
-Wire Wire Line
-	2600 5850 2700 5850
-Wire Wire Line
-	2600 6050 3400 6050
-Wire Wire Line
-	3000 5450 3000 6350
-Connection ~ 3000 6050
-Wire Wire Line
-	2700 6350 2600 6350
-Wire Wire Line
-	2600 5350 2600 5450
-$Comp
-L C C21
-U 1 1 5851837A
-P 2850 5450
-F 0 "C21" V 3102 5450 50  0000 C CNN
-F 1 "0.1uF" V 3011 5450 50  0000 C CNN
-F 2 "Capacitors_SMD:C_0805_HandSoldering" H 2888 5300 50  0001 C CNN
-F 3 "" H 2850 5450 50  0000 C CNN
-	1    2850 5450
-	0    -1   -1   0
-$EndComp
-Wire Wire Line
-	2600 5450 2700 5450
-Connection ~ 3000 5850
-$Comp
-L DB9 J3
-U 1 1 585187B1
-P 3650 6750
-F 0 "J3" H 3829 6796 50  0000 L CNN
-F 1 "DB9" H 3829 6705 50  0000 L CNN
-F 2 "mstock-pretty:DB9F" H 3650 6750 50  0001 C CNN
-F 3 "" H 3650 6750 50  0000 C CNN
-	1    3650 6750
-	1    0    0    -1
-$EndComp
-NoConn ~ 3200 6450
-NoConn ~ 3200 6550
-NoConn ~ 3200 7050
-NoConn ~ 3200 7150
-Wire Wire Line
-	3000 6350 3200 6350
-Connection ~ 3000 6350
-Wire Wire Line
-	2600 6750 3200 6750
-Wire Wire Line
-	2600 6850 3200 6850
-Wire Wire Line
-	2600 6650 3200 6650
-Wire Wire Line
-	2600 6550 3100 6550
-Wire Wire Line
-	3100 6550 3100 6950
-Wire Wire Line
-	3100 6950 3200 6950
-Text Label 1400 6750 2    60   ~ 0
-Serial0_RX
-Text Label 1400 6550 2    60   ~ 0
-Serial0_TX
-Text Label 1400 6850 2    60   ~ 0
-Serial0_CTS
-Text Label 1400 6650 2    60   ~ 0
-Serial0_RTS
-$Comp
 L R R17

Commit message: kicad updates
Parts:
- BT1: symbol Battery-RESCUE-soc -> Device:Battery
- C1, C10, C11, C12, C14, C15, C3, C4, C7, C8: symbol CP -> Device:CP
- C13, C16, C17, C18, C2, C24, C25, C5, C6, C9: symbol C -> Device:C
- D1, D2, D3, D4: symbol Led_Small -> Device:LED_Small
- J1, J4: symbol JACK_TRS_3PINS -> mstock:JACK_TRS_3PINS
- J2: symbol Mini_DIN-6 -> mstock:Mini_DIN-6
- J5: symbol JACK_TRRS_4PINS -> mstock:JACK_TRRS_4PINS
- L1, L2: symbol INDUCTOR -> Device:L
- P1: symbol CONN_02X08 -> Connector_Generic:Conn_02x08_Odd_Even
- P2: symbol ALTERA_DE1_GPIO -> mstock:ALTERA_DE1_GPIO
- P3: symbol CONN_02X06 -> Connector_Generic:Conn_02x06_Odd_Even
- R1, R10, R11, R12, R13, R14, R15, R16, R17, R18, R19, R2, R20, R3, R4, R5, R6, R7, R8, R9: symbol R -> Device:R
- U1: symbol SSM2603 -> mstock:SSM2603
- U2: symbol DS3234 -> mstock:DS3234
- U3: symbol speakjet -> mstock:speakjet
Connections:
- wire segments 144 -> 205

Commit message: update schematic
Parts:
- removed R13, R14: 10k, Resistors_SMD:R_0805_HandSoldering, symbol Device:R
- removed U3: speakjet, Housings_DIP:DIP-18_W7.62mm, symbol mstock:speakjet
- BT1: symbol Device:Battery -> device:Battery
- C1, C10, C11, C12, C14, C15, C3, C4, C7, C8: symbol Device:CP -> device:CP
- C13, C16, C17, C18, C2, C24, C25, C5, C6, C9: symbol Device:C -> device:C
- D1, D2, D3, D4: symbol Device:LED_Small -> device:LED_Small
- L1, L2: symbol Device:L -> device:L
- P1: symbol Connector_Generic:Conn_02x08_Odd_Even -> Connector:Conn_02x08_Odd_Even
- P3: symbol Connector_Generic:Conn_02x06_Odd_Even -> Connector:Conn_02x06_Odd_Even
- R1, R10, R11, R12, R15, R16, R17, R18, R19, R2, R20, R3, R4, R5, R6, R7, R8, R9: symbol Device:R -> device:R
Connections:
- net labels removed: Serial1_busy, speaking, voice
- wire segments 205 -> 178
- no-connect marks 9 -> 8
