File: 7seg/7seg.kicad_pcb (KiCad board)
At the start: 2 copper layers, 110.5 x 43.2 mm, 26 parts, among them IC1 ATTINY88-AZ, P1 TST, P2 TST, P3 SPI, P4 TST, P5 TST, Q1 MBT3904DW1, Q10 MBT3904DW1, Q2 MBT3904DW1, Q3 MBT3904DW1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

Commit message: spin 7seg board and io 2.5
Parts:
- moved Q1 24.1 mm to (124.5, 97.2)
- moved Q6 24.1 mm to (124.5, 115.6)
- moved Q10 17.2 mm to (124.5, 79.4)
- moved Q5 15.9 mm to (134.6, 79.4), turned to 0 degrees
- moved Q2 14.0 mm to (124.5, 87.6)
- moved Q7 14.0 mm to (124.5, 106.7)
- moved Q3 11.7 mm to (134.6, 87.6)
- moved Q8 11.7 mm to (134.6, 106.7)
- moved U1 3.18 mm to (174.6, 106.7)
- moved C3 3.17 mm to (168.3, 106.7)
- moved C2 2.62 mm to (182.2, 83.8)
- moved IC1 2.62 mm to (174.0, 84.5)
- moved P3 2.29 mm to (184.2, 102.2)
- moved RP1 2.01 mm to (163.2, 97.2), turned to 0 degrees
- moved RP2 1.91 mm to (163.2, 106.7)
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Routing:
- net +5V: track 0.00 -> 224.6 mm, vias 0 -> 3
- net Net-(D1-Pad15): track 0.00 -> 131.8 mm, vias 0 -> 2
- net Net-(D1-Pad3): track 0.00 -> 114.2 mm, vias 0 -> 1
- net Net-(D1-Pad16): track 0.00 -> 111.5 mm
- net Net-(D1-Pad12): track 0.00 -> 109.0 mm
- net Net-(D1-Pad11): track 0.00 -> 106.4 mm
- net Net-(D3-Pad4): track 0.00 -> 106.1 mm
- net Net-(D1-Pad13): track 0.00 -> 105.8 mm
- net Net-(D1-Pad14): track 0.00 -> 105.5 mm
- net Net-(D1-Pad5): track 0.00 -> 101.3 mm
- net Net-(D1-Pad7): track 0.00 -> 97.9 mm, vias 0 -> 1
- net Net-(D1-Pad10): track 0.00 -> 88.8 mm, vias 0 -> 1
- net /Digit9: track 0.00 -> 87.4 mm
- net Net-(D1-Pad9): track 0.00 -> 85.4 mm
- net /Digit12: track 0.00 -> 85.0 mm
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Other:
- board size 110.5 x 43.2 mm -> 109.2 x 45.7 mm

Commit message: Improve the silkscreen if we ever make more of these
Other:
- board text added: "+5V"
- board text added: "GND"
- board text added: "MISO"
- board text added: "MOSI"
- board text added: "SCK"
- board text added: "~RST"
- board text added: "~SS"
Changed lines of the file:
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@@
     (area 81.204999 73.3375 190.575001 121.1075)
     (thickness 1.6)
-    (drawings 4)
+    (drawings 11)
     (tracks 868)
     (zones 0)
@@
   (title_block
     (title "7 segment module")
-    (date 2017-01-09)
-    (rev 1.0)
+    (date 2017-05-02)
+    (rev 1.1)
     (company "Bexkat Systems LLC")
   )
@@
     (tags "QFP 0.8")
     (attr smd)
-    (fp_text reference IC1 (at 3.81 6.35) (layer B.SilkS)
+    (fp_text reference IC1 (at 0.254 -6.35) (layer B.SilkS)
       (effects (font (size 1 1) (thickness 0.15)) (justify mirror))
     )
@@
     (descr "Through hole pin header")
     (tags "pin header")
-    (fp_text reference P3 (at 0 5.1) (layer B.SilkS)
-      (effects (font (size 1 1) (thickness 0.15)) (justify mirror))
-    )
-    (fp_text value SPI (at 0 3.1) (layer B.Fab)
+    (fp_text reference P3 (at 0 -12.827) (layer B.SilkS)
+      (effects (font (size 1 1) (thickness 0.15)) (justify mirror))
+    )
+    (fp_text value SPI (at -0.635 2.921) (layer B.SilkS)
       (effects (font (size 1 1) (thickness 0.15)) (justify mirror))
     )
@@
     )
   )
+  (gr_text GND (at 186.817 88.392 90) (layer B.SilkS)
+    (effects (font (size 1 1) (thickness 0.2)) (justify mirror))
+  )
+  (gr_text +5V (at 186.69 105.791 90) (layer B.SilkS)
+    (effects (font (size 1 1) (thickness 0.2)) (justify mirror))
+  )
+  (gr_text MOSI (at 180.467 102.235) (layer B.SilkS)
+    (effects (font (size 1 1) (thickness 0.2)) (justify mirror))
+  )
+  (gr_text SCK (at 180.721 94.615) (layer B.SilkS)
+    (effects (font (size 1 1) (thickness 0.2)) (justify mirror))
+  )
+  (gr_text MISO (at 180.467 92.075) (layer B.SilkS)
+    (effects (font (size 1 1) (thickness 0.2)) (justify mirror))
+  )
+  (gr_text ~RST (at 180.848 97.282) (layer B.SilkS)
+    (effects (font (size 1 1) (thickness 0.2)) (justify mirror))
+  )
+  (gr_text ~SS (at 181.229 99.822) (layer B.SilkS)
+    (effects (font (size 1 1) (thickness 0.2)) (justify mirror))
+  )
   (gr_line (start 190.5 120.015) (end 81.28 120.015) (angle 90) (layer Edge.Cuts) (width 0.15))
