File: 7seg/7seg.sch (KiCad schematic (older format))
At the start: 26 parts, among them IC1 ATTINY88-AZ, P1 TST, P2 TST, P3 SPI, P4 TST, P5 TST, Q1 MBT3904DW1, Q10 MBT3904DW1, Q2 MBT3904DW1, Q3 MBT3904DW1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

Commit message: kicad updates
Parts:
- C2, C3: symbol C -> device:C
- D1, D2, D3, D4: symbol Quad7seg -> mstock:Quad7seg
- IC1: symbol ATTINY88-AZ -> atmel:ATTINY88-AU
- P1, P2, P4, P5: symbol TST -> Connector:Test_Point
- P3: symbol CONN_02X05 -> Connector:Conn_02x05_Odd_Even
- Q1, Q2, Q3, Q4, Q5, Q6, Q7, Q8, Q9: footprint mstock-new:SOT-363 -> mstock:SOT-363; symbol MBT3904DW1 -> mstock:MBT3904DW1
- Q10: symbol MBT3904DW1 -> mstock:MBT3904DW1
- RP1, RP2, RP3: footprint mstock-new:CAY16-J4 -> mstock:CAY16-J4; symbol R_PACK4 -> device:R_Pack04
- U1: symbol TLC6C5912 -> mstock:TLC6C5912
Connections:
- wire segments 112 -> 149
- no-connect marks 7 -> 14
